File: alarm_clock.sch (EAGLE design)
At the start: 27 parts, among them IC1 DS1307, U1 ATMEGA328P-PU

Commit message: In progress save/commit:
Parts:
- removed PH1: A1050_09, photo-elements:A1050_09
- added C5: 1uF, rcl:C-EU025-024X044
- added PH2: A1050_09, photo-elements:A1050_09
- added U2: MC14489BPE, MC14489BPE:MC14489BPE
- C1, C2: value (none) -> 22pF
- C3: value (none) -> 1uF
- C4: value (none) -> 330uF
- Q1: value (none) -> 16MHz
- R1: value (none) -> 10kΩ
- R2, R3, R4, R6, R7: value (none) -> 220Ω
- R8: value (none) -> 10KΩ
Connections:
- removed net N$1 (its old number): IC1.SCL, R7.2
- removed net N$10: D1.G, D2.G, D3.G, D4.G
- removed net N$11: D2.CK2
- removed net N$12: D3.CK2
- removed net N$13: D1.CK2
- removed net N$15: R3.2
- removed net N$17: R5.1
- removed net N$20: D1.DP
- removed net N$23: D2.DP
- removed net N$24: D3.DP
- removed net N$25: D4.DP
- removed net N$4 (its old number): D1.B, D2.B, D3.B, D4.B
- removed net N$5: D1.C, D2.C, D3.C, D4.C
- removed net N$6: D1.D, D2.D, D3.D, D4.D
- removed net N$7: D1.E, D2.E, D3.E, D4.E
- removed net N$8: D4.CK2
- removed net N$9: D1.F, D2.F, D3.F, D4.F
- new net A: D1.A, D2.A, D3.A, D4.A, LED1.A, LED2.A, U2.A
- new net B: D1.B, D2.B, D3.B, D4.B, LED3.A, U2.B
- new net C: D1.C, D2.C, D3.C, D4.C, U2.C
- new net CLK: U1.PD7, U2.CLK
- new net D: D1.D, D2.D, D3.D, D4.D, U2.D
- new net D1: D1.CK2, U2.BANK_1
- new net D2: D2.CK2, U2.BANK_2
- new net D3: D3.CK2, U2.BANK_3
- new net D4: D4.CK2, U2.BANK_4
- new net DATA: U1.PB0
- new net E: D1.E, D2.E, D3.E, D4.E, U2.E
- new net EN: U1.PD4, U2.~EN
- new net F: D1.F, D2.F, D3.F, D4.F, U2.F
- new net G: D1.G, D2.G, D3.G, D4.G, U2.G
- new net LEDS: LED1.C, LED2.C, LED3.C, U2.BANK_5
- new net P: D1.DP, D2.DP, D3.DP, D4.DP, U2.H
- new net PZ: R5.1, U1.PD3
- new net RX: R3.2, U2.RX
- new net SCL: IC1.SCL, R7.2, U1.PC5
- new net SDA: IC1.SDA, R6.2, U1.PC4
- new net SNZ: R4.1, U1.PD5
- new net VBAT: BATT.+, BATT.+1, C5.1, IC1.VBAT
- net GND: now also C3.2, C5.2, LED4.C, PH2.2, U1.GND_2, U2.VSS; no longer PH1.2
- net N$18: now also U1.PB7
- net N$19: now also U1.PB6
- net N$2: now also LED4.A, R4.2; no longer IC1.SDA, R6.2
- net N$21: now also PH2.1; no longer PH1.1
- net N$3: now also U2.DATA_IN; no longer D1.A, D2.A, D3.A, D4.A
- net VCC: now also C3.1, U1.AVCC, U2.VDD; no longer BATT.+, BATT.+1
Other:
- note added: "Input: Ambient Light Sensor"
- note added: "Logic: LED Display Driver"
- note added: "Logic: Microcontroller"
- note added: "Output: Alarm/Snooze - Piezo Buzzer"
- note added: "Output: Snooze - Large Red LED"
- note added: "Output: Time Display - 7-Seg LED"
- note added: "Output: Time Separators - Orange LED Alarm Set Indicator - Green LED"
- note added: "Power: Backup Battery"
- note added: "Time Control: Real Time Clock"
- moved on the sheet: BATT, C1, C2, C3, C4, D1, D2, D3, D4, D5, IC1, LED1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

Commit message: in progress commit:
Parts:
- added ALARM: (no value), switch:320-916
- added J1: USB-MICROB", SparkFun-Connectors:USB-MICROB"
- added S2, SNOOZE: (no value), switch-omron:10-XX
- R5: value (none) -> 1.5kΩ
Connections:
- new net N$5: ALARM.O, U1.PC0
- new net N$6: ALARM.S, U1.PC1
- new net N$9: SNOOZE.P, SNOOZE.P1, U1.PC2
- new net RESET: S2.P, U1.PC6
- net GND: now also ALARM.P, J1.GND, S2.S, S2.S1, SNOOZE.S, SNOOZE.S1
- net N$14: now also R8.E; no longer R8.A
- net SCL: now also U1.PC4; no longer U1.PC5
- net SDA: now also U1.PC5; no longer U1.PC4
- net VCC: now also J1.VBUS
Other:
- note added: "Logic: Microcontroller LED Display Driver"
- note added: "Power: Micro-USB power supply"
- note removed: "Logic: LED Display Driver"
- note removed: "Logic: Microcontroller"
- moved on the sheet: BATT, C1, C2, C3, C4, C5, D1, D2, D3, D4, D5, IC1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
